Commit message: feat: refine workcell layout and load official crx meshes

File: frontend/assets/robot/crx20ial/robot.urdf (robot description, URDF)
Before this commit: robot crx20ial_urdf_demo, 8 links, 7 joints
Links:
- removed link link_1
- removed link link_2
- removed link link_3
- removed link link_4
- removed link link_5
- removed link link_6
- removed link tool0
- added link J1_link; visual mesh filename=meshes/crx20ial/visual/j1.dae
- added link J2_link; visual mesh filename=meshes/crx20ial/visual/j2.dae
- added link J3_link; visual mesh filename=meshes/crx20ial/visual/j3.dae
- added link J4_link; visual mesh filename=meshes/crx20ial/visual/j4.dae
- added link J5_link; visual mesh filename=meshes/crx20ial/visual/j5.dae
- added link J6_link; visual mesh filename=meshes/crx20ial/visual/j6.dae
- added link ee_link
- added link flange
- added link world
- link base_link: geometry visual mesh filename=meshes/crx20ial/visual/base.dae
Joints:
- removed joint elbow_joint
- removed joint shoulder_lift_joint
- removed joint shoulder_pan_joint
- removed joint tool0_fixed
- removed joint wrist_1_joint
- removed joint wrist_2_joint
- removed joint wrist_3_joint
- added joint J1: type revolute, parent base_link, child J1_link, origin xyz=0 0 0.245 rpy=0 0 0, axis 0 0 1, limit lower=-3.139847 upper=3.139847 effort=750 velocity=1.396263
- added joint J2: type revolute, parent J1_link, child J2_link, origin xyz=0 0 0 rpy=0 0 0, axis 0 1 0, limit lower=-3.139847 upper=3.139847 effort=750 velocity=1.396263
- added joint J3: type revolute, parent J2_link, child J3_link, origin xyz=0 0 0.710 rpy=0 0 0, axis 0 -1 0, limit lower=-4.712389 upper=4.712389 effort=350 velocity=2.094395
- added joint J4: type revolute, parent J3_link, child J4_link, origin xyz=0 0 0 rpy=0 0 0, axis -1 0 0, limit lower=-3.316126 upper=3.316126 effort=150 velocity=1.963495
- added joint J5: type revolute, parent J4_link, child J5_link, origin xyz=0.540 0 0 rpy=0 0 0, axis 0 -1 0, limit lower=-3.139847 upper=3.139847 effort=110 velocity=1.570796
- added joint J6: type revolute, parent J5_link, child J6_link, origin xyz=0 -0.150 0 rpy=0 0 0, axis -1 0 0, limit lower=-3.926991 upper=3.926991 effort=110 velocity=1.963495
- added joint J6-flange: type fixed, parent J6_link, child flange, origin xyz=0.160 0 0 rpy=0 0 0
- added joint base_joint: type fixed, parent world, child base_link, origin xyz=0 0 0.75 rpy=0 0 0
- added joint child_joint: type fixed, parent flange, child ee_link, origin xyz=0 0 0 rpy=0 0 0
